File: audio_power_amplifier.kicad_sch (KiCad schematic)
At the start: 80 parts, among them Q1 BC546, Q10 BC546, Q11 BC546, Q12 BC546, Q13 MJE15035, Q14 BC546, Q15 MJE15034, Q16 MJE15035, Q17 MJL4302, Q18 MJL4281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

Commit message: cosmetics
Other:
- note added: "Left Channel"
- note added: "Right Channel"
- title: Stereo Audio Power Amplifier -> Audio Power Amplifier
- moved on the sheet: C1, C10, C11, C12, C13, C14, C15, C16, C17, C18, C19, C2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
